File: micro.kicad_sch (KiCad schematic)
At the start: 24 parts, among them U1 ${ALTIUM_VALUE}, X1 ${ALTIUM_VALUE}, X2 ${ALTIUM_VALUE}

Commit message: ultimas dos clases - anyadidas mas footprints mas esquematico
Parts:
- U1: footprint (none) -> wearable_footprints:QFN40P600X600X90-49N-D
Changed lines of the file:
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@@
 			)
 		)
-		(property "Footprint" ""
+		(property "Footprint" "wearable_footprints:QFN40P600X600X90-49N-D"
 			(at 81.28 123.19 0)
 			(effects
